Commit message: feat(microbot): add AprilTag-following stack for the 2WD vehicle
Bring the ESP32 differential-drive bot to life in ROS 2: stream the
ESP32-CAM feed into ROS, detect and visualize AprilTags, drive the robot
from wheel encoders in RViz, and follow a tag with a tuning-free (no-PID)
controller.

New microbot_description nodes:
- camera_stream: bridge the ESP32-CAM MJPEG HTTP stream to /camera/image_raw.
- apriltag_detector: detect tags (cv2.aruco) and publish an annotated
  /apriltag/image for RViz.
- apriltag_follower: no-PID follower publishing /cmd_vel. Distance
  bang-bang (forward / hold / ease-back) with a wide center deadband. Arc
  turns are gated by max_turn (currently 0 = straight only) and a small
  straight_bias trims the drivetrain's right-drift. Stops in place when the
  tag leaves the frame.
- wheel_odometry: integrate /joint_states encoder angles into /odom and the
  odom->base_link TF; encoder_direction=-1 corrects the sign so forward
  driving reads as forward in RViz.
- joint_states, camera_viz: supporting wheel-angle and camera-aggregate viz.

Launch:
- hardware.launch.py: real-robot view (robot_state_publisher, odometry,
  camera stream, detection, RViz).
- follow.launch.py: run the follower with tunable args (desired_distance,
  forward_speed, max_turn, center_deadband, straight_bias, wheel_min, tag_id).

Also: register entry points in setup.py, add package.xml deps, add wheel
joints to the URDF, extend the RViz config, trim behaviors.launch.py,
include the standalone apriltag_follower reference scripts, and gitignore
the auto-generated MUJOCO_LOG.TXT.

File: src/02_micro_ros/microbot_description/urdf/microbot.urdf.xacro (robot description, xacro)
@@ -100,4 +100,17 @@
   <xacro:ultrasonic name="us_left"  px="0"            py="${ body_y/2}" pz="0" yaw="1.5708"/>
   <xacro:ultrasonic name="us_right" px="0"            py="${-body_y/2}" pz="0" yaw="-1.5708"/>
+  <!-- ===================== camera (ESP32-CAM), front-facing ===================== -->
+  <link name="camera_link">
+    <visual>
+      <geometry><box size="0.03 0.03 0.02"/></geometry>
+      <material name="black"/>
+    </visual>
+    <xacro:box_inertial mass="0.02" x="0.03" y="0.03" z="0.02"/>
+  </link>
+  <joint name="camera_joint" type="fixed">
+    <parent link="base_link"/>
+    <child link="camera_link"/>
+    <origin xyz="${body_x/2} 0 ${body_z/2+0.03}" rpy="0 0 0"/>
+  </joint>
   <!-- ===================== labelled components ===================== -->
   <xacro:part name="battery" x="0.10" y="0.12" z="0.04" px="-0.05" py="0"     pz="${body_z/2+0.02}" material="bat_green"/>
